Commit message: CT controller updated

File: urdf/wheel.urdf.xacro (robot description, xacro)
@@ -39,7 +39,7 @@
 			<parent link="${prefix}_wheelActuator"/>
 			<child  link="${prefix}_wheel"/>
-			<limit effort="5" velocity="30"/>  <!-- effort limit in N (prismatic) or N.m (revolute), Velocity limit in m/s or rad/s -->
+			<limit effort="3" velocity="20"/>  <!-- effort limit in N (prismatic) or N.m (revolute), Velocity limit in m/s or rad/s -->
 			<axis xyz="0 1 0"/>
-			<joint_properties damping="0.1" friction="0.0"/>
+			<joint_properties damping="0.4830" friction="0.0011"/>
 		</joint>
     		<!--transmission name="Diff_${prefix}_wheel_trans">
