Commit message: robot_localization added

File: urdf/Igor.urdf.xacro (robot description, xacro)
@@ -127,4 +127,32 @@
 		<origin xyz="${0.02} ${(actuator_y_size/2)+wheel_length/2} 0.0" rpy="0 0 0" />
 	</xacro:igor_wheel>
+	<!--Right wheel actuator imu_link for getting data in imu frame -->
+    	<link name="RwheelActuator_imu_link"/>
+	<joint name="RwheelActuator_imu_link" type="fixed">
+		<origin xyz="0 0 0" rpy="${M_PI/2} ${M_PI/2} 0" />
+		<parent link="R_wheelActuator" />
+	        <child link="RwheelActuator_imu_link" />
+	</joint>
+	<!--Left wheel actuator imu_link for getting data in imu frame -->
+    	<link name="LwheelActuator_imu_link"/>
+	<joint name="LwheelActuator_imu_link" type="fixed">
+		<origin xyz="0 0 0" rpy="${-M_PI/2} ${M_PI/2} ${0}" />
+		<parent link="L_wheelActuator" />
+	        <child link="LwheelActuator_imu_link" />
+	</joint>
+	<!--Left hip actuator imu_link for getting data in imu frame -->
+    	<link name="LhipActuator_imu_link"/>
+	<joint name="LhipActuator_imu_link" type="fixed">
+		<origin xyz="0 0 0" rpy="${-M_PI/2} ${0} ${0}" />
+		<parent link="L_baseActuator" />
+	        <child link="LhipActuator_imu_link" />
+	</joint>
+	<!--Right hip actuator imu_link for getting data in imu frame -->
+    	<link name="RhipActuator_imu_link"/>
+	<joint name="RhipActuator_imu_link" type="fixed">
+		<origin xyz="0 0 0" rpy="${M_PI/2} ${0} ${0}" />
+		<parent link="R_baseActuator" />
+	        <child link="RhipActuator_imu_link" />
+	</joint>
 	<!--Robot Center Dummy-->
 	<link name="robot_center_link">

File: urdf/lowerleg.urdf.xacro (robot description, xacro)
@@ -27,5 +27,5 @@
 			<parent link="${prefix}_kneeActuator"/>
 			<child  link="${prefix}_lowerleg"/>
-			<limit effort="15" lower="0" upper="2" velocity="10"/>
+			<limit effort="15" lower="0" upper="0" velocity="10"/>
 			<axis xyz="0 1 0"/>
 			<dynamics damping="0.1"/>

File: urdf/upperleg.urdf.xacro (robot description, xacro)
@@ -29,5 +29,5 @@
 			<parent link="${prefix}_baseActuator"/>
 			<child  link="${prefix}_upperleg"/>
-			<limit effort="${15}" lower="-2" upper="2" velocity="10"/>
+			<limit effort="${15}" lower="-0" upper="0" velocity="10"/>
 			<axis xyz="0 1 0"/>
 			<dynamics damping="0.1"/>

Commit message: Updated

File: urdf/Igor.urdf.xacro (robot description, xacro)
@@ -9,5 +9,5 @@
 	<xacro:property name="base_y_size" value="0.3048" />
 	<xacro:property name="base_x_size" value="0.127" />
-	<xacro:property name="base_z_size" value="0.3048" />
+	<xacro:property name="base_z_size" value="0.22" />
 	<xacro:property name="base_y_offset" value="0.0076" />
 		  <!-- Actuator Size -->

File: urdf/Igor_knee.urdf.xacro (robot description, xacro)
@@ -7,7 +7,7 @@
 	<xacro:include filename="$(find igor)/urdf/lowerleg.urdf.xacro" />
 	  <!-- Base Size -->
-	<xacro:property name="base_y_size" value="0.3048" />
-	<xacro:property name="base_x_size" value="0.127" />
-	<xacro:property name="base_z_size" value="0.3048" />
+	<xacro:property name="base_y_size" value="0.305" />
+	<xacro:property name="base_x_size" value="0.09" />
+	<xacro:property name="base_z_size" value="0.218" />
 	<xacro:property name="base_y_offset" value="0.0076" />
 		  <!-- Actuator Size -->
@@ -40,6 +40,6 @@
   		<inertial>
      			<origin xyz="0 0 0" rpy="0.0 0.0 0.0" />
-			<mass value="5.0" />
-      			<inertia izz="0.04543" iyz="0.000" ixz="0.00000" iyy="0.04543" ixy="0.000" ixx="0.0774" />
+			<mass value="7.5" />
+      			<inertia izz="0.0632" iyz="0.000" ixz="0.00000" iyy="0.0347" ixy="0.000" ixx="0.0878" />
 		</inertial>
 			<!-- Mass change for uncertainity-->
@@ -50,5 +50,5 @@
 		</inertial-->
 		<visual>
-			<origin rpy="${M_PI} 0.0 ${-M_PI/2}" xyz="${base_x_size/2} ${base_y_size/2+base_y_offset} ${base_z_size/2}"/>
+			<origin rpy="${M_PI} 0.0 ${-M_PI/2}" xyz="${base_x_size/2} ${base_y_size/2+base_y_offset} ${base_z_size/1.4}"/>
 			<geometry>
 				<!--box size="0.30 0.1 0.30"/-->
@@ -86,44 +86,44 @@
 	<xacro:igor_actuator prefix="L_base" reflect="1" parent_link="chassis" flip="1">
                    <!--Origin of the joint from parent frame-->
-		<origin xyz="0.0 ${base_y_size/2+actuator_y_size/2} ${0}" rpy="${0} 0 ${0}" />
+		<origin xyz="${0.0} ${base_y_size/2+actuator_y_size/2} ${-0.06}" rpy="${0} 0 ${0}" />
 	</xacro:igor_actuator>
 	<xacro:igor_actuator prefix="R_base" reflect="-1" parent_link="chassis" flip="0">
-		<origin xyz="0.0 -${base_y_size/2+actuator_y_size/2} 0.0" rpy="0 0 0" />
+		<origin xyz="${0.0} -${base_y_size/2+actuator_y_size/2} ${-0.06}" rpy="0 0 0" />
 	</xacro:igor_actuator>
 	<!--Right Leg-->
 	<xacro:upperLeg prefix="R" reflect="-1" flip="1">
-		<origin xyz="${upper_leg_radius} -${actuator_y_size/2+upper_leg_radius} 0.0" rpy="0 0 0" />
+		<origin xyz="${0} -${actuator_y_size/2+upper_leg_radius} 0.0" rpy="0 0 0" />
 	</xacro:upperLeg>
 	<xacro:lowerLeg prefix="R" reflect="-1" flip="1">
-		<origin xyz="${1.2*lower_leg_radius} ${actuator_y_size/2+lower_leg_radius} 0.0" rpy="0 0 0" />
+		<origin xyz="${0} ${actuator_y_size/2+lower_leg_radius} 0.0" rpy="0 0 0" />
 	</xacro:lowerLeg>
 	<!--Left Leg-->
 	<xacro:upperLeg prefix="L" reflect="1" flip="0">
-		<origin xyz="${upper_leg_radius} ${actuator_y_size/2+upper_leg_radius} 0.0" rpy="0 0 0" />
+		<origin xyz="${0} ${actuator_y_size/2+upper_leg_radius} 0.0" rpy="0 0 0" />
 	</xacro:upperLeg>
 	<xacro:lowerLeg prefix="L" reflect="1" flip="0">
-		<origin xyz="${1.2*lower_leg_radius} -${actuator_y_size/2+lower_leg_radius} 0.0" rpy="0 0 0" />
+		<origin xyz="${0} -${actuator_y_size/2+lower_leg_radius} 0.0" rpy="0 0 0" />
 	</xacro:lowerLeg>
 	<!--Right knee-->
 	<xacro:igor_actuator prefix="R_knee" reflect="-1" parent_link="R_upperleg" flip="0">
-		<origin xyz="-${1.2*upper_leg_radius} ${actuator_y_size/2+upper_leg_radius} -${upper_leg_length+actuator_z_size/3}" rpy="0 0 0" />
+		<origin xyz="${0} ${actuator_y_size/2+upper_leg_radius} -${upper_leg_length+actuator_z_size/3}" rpy="0 0 0" />
 	</xacro:igor_actuator>
 	<!--Left knee-->
 	<xacro:igor_actuator prefix="L_knee" reflect="1" parent_link="L_upperleg" flip="1">
-		<origin xyz="-${1.2*upper_leg_radius} -${actuator_y_size/2+upper_leg_radius} -${upper_leg_length+actuator_z_size/3}" rpy="0 0 0" />
+		<origin xyz="${0} -${actuator_y_size/2+upper_leg_radius} -${upper_leg_length+actuator_z_size/3}" rpy="0 0 0" />
 	</xacro:igor_actuator>
 	<!--Right wheel-->
 	<xacro:igor_actuator prefix="R_wheel" reflect="-1" parent_link="R_lowerleg" flip="0">
-		<origin xyz="-${lower_leg_radius} -${actuator_y_size-0.0038} -${lower_leg_length+actuator_z_size/2.5}" rpy="0 0 0" />
+		<origin xyz="${0} -${actuator_y_size-0.0038} -${lower_leg_length+actuator_z_size/2.5}" rpy="0 0 0" />
 	</xacro:igor_actuator>
 	<xacro:igor_wheel prefix="R" flip="0" reflect="-1">
-		<origin xyz="${0.02} -${(actuator_y_size/2)+wheel_length/2} 0.0" rpy="0 0 0" />
+		<origin xyz="${0} -${(actuator_y_size/2)+wheel_length/2} 0.0" rpy="0 0 0" />
 	</xacro:igor_wheel>
 	<!--Left wheel-->
 	<xacro:igor_actuator prefix="L_wheel" reflect="1" parent_link="L_lowerleg" flip="1">
-		<origin xyz="-${lower_leg_radius} ${actuator_y_size-0.0038} -${lower_leg_length+actuator_z_size/2.5}" rpy="0 0 0" />
+		<origin xyz="${0} ${actuator_y_size-0.0038} -${lower_leg_length+actuator_z_size/2.5}" rpy="0 0 0" />
 	</xacro:igor_actuator>
 	<xacro:igor_wheel prefix="L" flip="1" reflect="1">
-		<origin xyz="${0.02} ${(actuator_y_size/2)+wheel_length/2} 0.0" rpy="0 0 0" />
+		<origin xyz="${0} ${(actuator_y_size/2)+wheel_length/2} 0.0" rpy="0 0 0" />
 	</xacro:igor_wheel>
 	<!--Robot Center Dummy-->
@@ -141,5 +141,5 @@
 	</link>
 	<joint name="actuator_to_robot_center" type="fixed">
-		<origin xyz="${0.02} -${base_y_size/2+actuator_y_size/2} 0.0" rpy="0 0 0" />
+		<origin xyz="${0} -${base_y_size/2+actuator_y_size/2} 0.0" rpy="0 0 0" />
 		<parent link="L_wheelActuator" />
 	        <child link="robot_center_link" />
@@ -197,5 +197,5 @@
 			<updateRate>500.0</updateRate>
 			<bodyName>robot_center_link</bodyName>
-			<topicName>center</topicName>
+			<topicName>centerOdom</topicName>
 			<gaussianNoise>0.0</gaussianNoise>
 			<frameName>map</frameName>
@@ -205,15 +205,15 @@
 	</gazebo>
 	<!-- Body IMU Sensor -->
-	<!--gazebo reference="chassis">
+	<gazebo reference="chassis">
 	    <gravity>true</gravity>
 	    <sensor name="body_imu" type="imu">
 	      <always_on>true</always_on>
 	      <visualize>true</visualize>
-	      <!topic>__default_topic__</topic>
+	      <!--topic>__default_topic__</topic-->
 	      <plugin filename="libgazebo_ros_imu_sensor.so" name="imu_plugin">
 		<robotNamespace>/igor</robotNamespace>
 		<topicName>body_imu/data</topicName>
 		<bodyName>chassis</bodyName>
-		<updateRateHZ>1000.0</updateRateHZ>
+		<updateRateHZ>500.0</updateRateHZ>
 		<gaussianNoise>0.0</gaussianNoise>
 		<xyzOffset>0 0 0</xyzOffset>
@@ -223,4 +223,4 @@
 	      <pose>0 0 0 0 0 0</pose>
 	    </sensor>
-	</gazebo-->
+	</gazebo>
 </robot>

File: urdf/actuator.urdf.xacro (robot description, xacro)
@@ -4,5 +4,5 @@
 		<link name="${prefix}Actuator">
 			<visual>
-				<origin rpy="${(flip*M_PI)+(M_PI/2)} ${M_PI} ${0}" xyz="${actuator_x_size/2} ${reflect*(-actuator_y_size/2)} ${reflect*(-actuator_z_size/2)}"/>
+				<origin rpy="${(flip*M_PI)+(M_PI/2)} ${M_PI} ${0}" xyz="${actuator_x_size/3} ${reflect*(-actuator_y_size/2)} ${reflect*(-actuator_z_size/2)}"/>
 				<geometry>
 					<mesh filename="package://igor/meshes/X8-Export.STL" scale="0.001 0.001 0.001"/>
@@ -20,5 +20,5 @@
 	    		<inertial>
 	      			<mass value="0.46"/>
-	      			<inertia ixx="0.00066" ixy="0.0" ixz="0.0" iyy="0.00054" iyz="0.0" izz="0.00028"/>
+	      			<inertia iyy="0.00066" ixy="0.0" ixz="0.0" izz="0.00054" iyz="0.0" ixx="0.00028"/>
 	    		</inertial>
 		</link>

Commit message: URDF updated

File: urdf/Igor.urdf.xacro (robot description, xacro)
@@ -7,7 +7,7 @@
 	<xacro:include filename="$(find igor)/urdf/lowerleg.urdf.xacro" />
 	  <!-- Base Size -->
-	<xacro:property name="base_y_size" value="0.3048" />
-	<xacro:property name="base_x_size" value="0.127" />
-	<xacro:property name="base_z_size" value="0.22" />
+	<xacro:property name="base_y_size" value="0.305" />
+	<xacro:property name="base_x_size" value="0.09" />
+	<xacro:property name="base_z_size" value="0.218" />
 	<xacro:property name="base_y_offset" value="0.0076" />
 		  <!-- Actuator Size -->
@@ -40,6 +40,6 @@
   		<inertial>
      			<origin xyz="0 0 0" rpy="0.0 0.0 0.0" />
-			<mass value="5.0" />
-      			<inertia izz="0.04543" iyz="0.000" ixz="0.00000" iyy="0.04543" ixy="0.000" ixx="0.0774" />
+			<mass value="7.5" />
+      			<inertia izz="0.0632" iyz="0.000" ixz="0.00000" iyy="0.0347" ixy="0.000" ixx="0.0878" />
 		</inertial>
 			<!-- Mass change for uncertainity-->
@@ -50,5 +50,5 @@
 		</inertial-->
 		<visual>
-			<origin rpy="${M_PI} 0.0 ${-M_PI/2}" xyz="${base_x_size/2} ${base_y_size/2+base_y_offset} ${base_z_size/2}"/>
+			<origin rpy="${M_PI} 0.0 ${-M_PI/2}" xyz="${base_x_size/2} ${base_y_size/2+base_y_offset} ${base_z_size/1.4}"/>
 			<geometry>
 				<!--box size="0.30 0.1 0.30"/-->
@@ -86,44 +86,44 @@
 	<xacro:igor_actuator prefix="L_base" reflect="1" parent_link="chassis" flip="1">
                    <!--Origin of the joint from parent frame-->
-		<origin xyz="0.0 ${base_y_size/2+actuator_y_size/2} ${0}" rpy="${0} 0 ${0}" />
+		<origin xyz="0.0 ${base_y_size/2+actuator_y_size/2} ${-0.06}" rpy="${0} 0 ${0}" />
 	</xacro:igor_actuator>
 	<xacro:igor_actuator prefix="R_base" reflect="-1" parent_link="chassis" flip="0">
-		<origin xyz="0.0 -${base_y_size/2+actuator_y_size/2} 0.0" rpy="0 0 0" />
+		<origin xyz="0.0 -${base_y_size/2+actuator_y_size/2} ${-0.06}" rpy="0 0 0" />
 	</xacro:igor_actuator>
 	<!--Right Leg-->
 	<xacro:upperLeg prefix="R" reflect="-1" flip="1">
-		<origin xyz="${upper_leg_radius} -${actuator_y_size/2+upper_leg_radius} 0.0" rpy="0 0 0" />
+		<origin xyz="${0} -${actuator_y_size/2+upper_leg_radius} 0.0" rpy="0 0 0" />
 	</xacro:upperLeg>
 	<xacro:lowerLeg prefix="R" reflect="-1" flip="1">
-		<origin xyz="${1.2*lower_leg_radius} ${actuator_y_size/2+lower_leg_radius} 0.0" rpy="0 0 0" />
+		<origin xyz="${0} ${actuator_y_size/2+lower_leg_radius} 0.0" rpy="0 0 0" />
 	</xacro:lowerLeg>
 	<!--Left Leg-->
 	<xacro:upperLeg prefix="L" reflect="1" flip="0">
-		<origin xyz="${upper_leg_radius} ${actuator_y_size/2+upper_leg_radius} 0.0" rpy="0 0 0" />
+		<origin xyz="${0} ${actuator_y_size/2+upper_leg_radius} 0.0" rpy="0 0 0" />
 	</xacro:upperLeg>
 	<xacro:lowerLeg prefix="L" reflect="1" flip="0">
-		<origin xyz="${1.2*lower_leg_radius} -${actuator_y_size/2+lower_leg_radius} 0.0" rpy="0 0 0" />
+		<origin xyz="${0} -${actuator_y_size/2+lower_leg_radius} 0.0" rpy="0 0 0" />
 	</xacro:lowerLeg>
 	<!--Right knee-->
 	<xacro:igor_actuator prefix="R_knee" reflect="-1" parent_link="R_upperleg" flip="0">
-		<origin xyz="-${1.2*upper_leg_radius} ${actuator_y_size/2+upper_leg_radius} -${upper_leg_length+actuator_z_size/3}" rpy="0 0 0" />
+		<origin xyz="${0} ${actuator_y_size/2+upper_leg_radius} -${upper_leg_length+actuator_z_size/3}" rpy="0 0 0" />
 	</xacro:igor_actuator>
 	<!--Left knee-->
 	<xacro:igor_actuator prefix="L_knee" reflect="1" parent_link="L_upperleg" flip="1">
-		<origin xyz="-${1.2*upper_leg_radius} -${actuator_y_size/2+upper_leg_radius} -${upper_leg_length+actuator_z_size/3}" rpy="0 0 0" />
+		<origin xyz="${0} -${actuator_y_size/2+upper_leg_radius} -${upper_leg_length+actuator_z_size/3}" rpy="0 0 0" />
 	</xacro:igor_actuator>
 	<!--Right wheel-->
 	<xacro:igor_actuator prefix="R_wheel" reflect="-1" parent_link="R_lowerleg" flip="0">
-		<origin xyz="-${lower_leg_radius} -${actuator_y_size-0.0038} -${lower_leg_length+actuator_z_size/2.5}" rpy="0 0 0" />
+		<origin xyz="${0} -${actuator_y_size-0.0038} -${lower_leg_length+actuator_z_size/2.5}" rpy="0 0 0" />
 	</xacro:igor_actuator>
 	<xacro:igor_wheel prefix="R" flip="0" reflect="-1">
-		<origin xyz="${0.02} -${(actuator_y_size/2)+wheel_length/2} 0.0" rpy="0 0 0" />
+		<origin xyz="${0.0} -${(actuator_y_size/2)+wheel_length/2} 0.0" rpy="0 0 0" />
 	</xacro:igor_wheel>
 	<!--Left wheel-->
 	<xacro:igor_actuator prefix="L_wheel" reflect="1" parent_link="L_lowerleg" flip="1">
-		<origin xyz="-${lower_leg_radius} ${actuator_y_size-0.0038} -${lower_leg_length+actuator_z_size/2.5}" rpy="0 0 0" />
+		<origin xyz="${0} ${actuator_y_size-0.0038} -${lower_leg_length+actuator_z_size/2.5}" rpy="0 0 0" />
 	</xacro:igor_actuator>
 	<xacro:igor_wheel prefix="L" flip="1" reflect="1">
-		<origin xyz="${0.02} ${(actuator_y_size/2)+wheel_length/2} 0.0" rpy="0 0 0" />
+		<origin xyz="${0.0} ${(actuator_y_size/2)+wheel_length/2} 0.0" rpy="0 0 0" />
 	</xacro:igor_wheel>
 	<!--Right wheel actuator imu_link for getting data in imu frame -->
@@ -156,5 +156,5 @@
 	</joint>
 	<!--Robot Center Dummy-->
-	<link name="robot_center_link">
+	<!--link name="robot_center_link">
   		<inertial>
      			<origin xyz="0 0 0" rpy="0.0 0.0 0.0" />
@@ -169,5 +169,5 @@
 	</link>
 	<joint name="actuator_to_robot_center" type="fixed">
-		<origin xyz="${0.02+0.15*0} -${base_y_size/2+actuator_y_size/2} 0.0" rpy="0 0 0" />
+		<origin xyz="${0} -${base_y_size/2+actuator_y_size/2} 0.0" rpy="0 0 0" />
 		<parent link="L_wheelActuator" />
 	        <child link="robot_center_link" />
@@ -175,7 +175,7 @@
 	<gazebo reference="actuator_to_robot_center">
   		<preserveFixedJoint>true</preserveFixedJoint>
-	</gazebo>
+	</gazebo-->
 	<!-- Odometery Sensor -->
-	<gazebo>
+	<!--gazebo>
 		<plugin name="p3d_base_controller" filename= "libgazebo_ros_p3d.so">
 			<robotNamespace>/igor</robotNamespace>
@@ -189,7 +189,7 @@
 			<rpyOffsets>0 0 0</rpyOffsets>
 		</plugin>
-	</gazebo>
+	</gazebo-->
 	<!-- IMU Sensor -->
-	<gazebo reference="chassis">
+	<!--gazebo reference="chassis">
 	    <gravity>true</gravity>
 	    <sensor name="imu_sensor" type="imu">
@@ -209,4 +209,4 @@
 	      <pose>0 0 0 0 0 0</pose>
 	    </sensor>
-	</gazebo>
+	</gazebo-->
 </robot>

Commit message: Damping coefficient added

File: urdf/Igor.urdf.xacro (robot description, xacro)
@@ -117,5 +117,5 @@
 		<origin xyz="${0} -${actuator_y_size-0.0038} -${lower_leg_length+actuator_z_size/2.5}" rpy="0 0 0" />
 	</xacro:igor_actuator>
-	<xacro:igor_wheel prefix="R" flip="0" reflect="-1">
+	<xacro:igor_wheel prefix="R" flip="0" reflect="-1" damping="0.25">
 		<origin xyz="${0.0} -${(actuator_y_size/2)+wheel_length/2} 0.0" rpy="0 0 0" />
 	</xacro:igor_wheel>
@@ -124,5 +124,5 @@
 		<origin xyz="${0} ${actuator_y_size-0.0038} -${lower_leg_length+actuator_z_size/2.5}" rpy="0 0 0" />
 	</xacro:igor_actuator>
-	<xacro:igor_wheel prefix="L" flip="1" reflect="1">
+	<xacro:igor_wheel prefix="L" flip="1" reflect="1" damping="0.25">
 		<origin xyz="${0.0} ${(actuator_y_size/2)+wheel_length/2} 0.0" rpy="0 0 0" />
 	</xacro:igor_wheel>

File: urdf/Igor_knee.urdf.xacro (robot description, xacro)
@@ -117,5 +117,5 @@
 		<origin xyz="${0} -${actuator_y_size-0.0038} -${lower_leg_length+actuator_z_size/2.5}" rpy="0 0 0" />
 	</xacro:igor_actuator>
-	<xacro:igor_wheel prefix="R" flip="0" reflect="-1">
+	<xacro:igor_wheel prefix="R" flip="0" reflect="-1" damping="0.25">
 		<origin xyz="${0} -${(actuator_y_size/2)+wheel_length/2} 0.0" rpy="0 0 0" />
 	</xacro:igor_wheel>
@@ -124,5 +124,5 @@
 		<origin xyz="${0} ${actuator_y_size-0.0038} -${lower_leg_length+actuator_z_size/2.5}" rpy="0 0 0" />
 	</xacro:igor_actuator>
-	<xacro:igor_wheel prefix="L" flip="1" reflect="1">
+	<xacro:igor_wheel prefix="L" flip="1" reflect="1" damping="0.25">
 		<origin xyz="${0} ${(actuator_y_size/2)+wheel_length/2} 0.0" rpy="0 0 0" />
 	</xacro:igor_wheel>

File: urdf/wheel.urdf.xacro (robot description, xacro)
@@ -1,5 +1,5 @@
 <?xml version="1.0"?>
 <robot xmlns:xacro="http://ros.org/wiki/xacro" name="igor_wheel">
-	<xacro:macro name="igor_wheel" params="prefix flip reflect *joint_pose">
+	<xacro:macro name="igor_wheel" params="prefix flip reflect damping *joint_pose">
 		<link name="${prefix}_wheel">
 			<visual>
@@ -41,5 +41,5 @@
 			<limit effort="3" velocity="20"/>  <!-- effort limit in N (prismatic) or N.m (revolute), Velocity limit in m/s or rad/s -->
 			<axis xyz="0 1 0"/>
-			<joint_properties damping="0.4830" friction="0.0011"/>
+			<dynamics damping="${damping}" friction="0.0011"/>
 		</joint>
     		<!--transmission name="Diff_${prefix}_wheel_trans">

Commit message: Gains updated

File: urdf/Igor.urdf.xacro (robot description, xacro)
@@ -117,5 +117,5 @@
 		<origin xyz="${0} -${actuator_y_size-0.0038} -${lower_leg_length+actuator_z_size/2.5}" rpy="0 0 0" />
 	</xacro:igor_actuator>
-	<xacro:igor_wheel prefix="R" flip="0" reflect="-1" damping="0.25">
+	<xacro:igor_wheel prefix="R" flip="0" reflect="-1" damping="0.25" static_friction="0.0011">
 		<origin xyz="${0.0} -${(actuator_y_size/2)+wheel_length/2} 0.0" rpy="0 0 0" />
 	</xacro:igor_wheel>
@@ -124,5 +124,5 @@
 		<origin xyz="${0} ${actuator_y_size-0.0038} -${lower_leg_length+actuator_z_size/2.5}" rpy="0 0 0" />
 	</xacro:igor_actuator>
-	<xacro:igor_wheel prefix="L" flip="1" reflect="1" damping="0.25">
+	<xacro:igor_wheel prefix="L" flip="1" reflect="1" damping="0.25" static_friction="0.0011">
 		<origin xyz="${0.0} ${(actuator_y_size/2)+wheel_length/2} 0.0" rpy="0 0 0" />
 	</xacro:igor_wheel>

File: urdf/Igor_knee.urdf.xacro (robot description, xacro)
@@ -40,5 +40,5 @@
   		<inertial>
      			<origin xyz="0 0 0" rpy="0.0 0.0 0.0" />
-			<mass value="7.5" />
+			<mass value="${7.5}" />
       			<inertia izz="0.0632" iyz="0.000" ixz="0.00000" iyy="0.0347" ixy="0.000" ixx="0.0878" />
 		</inertial>
@@ -117,5 +117,5 @@
 		<origin xyz="${0} -${actuator_y_size-0.0038} -${lower_leg_length+actuator_z_size/2.5}" rpy="0 0 0" />
 	</xacro:igor_actuator>
-	<xacro:igor_wheel prefix="R" flip="0" reflect="-1" damping="${0.25}">
+	<xacro:igor_wheel prefix="R" flip="0" reflect="-1" damping="${0.17}" static_friction="0.0011">
 		<origin xyz="${0} -${(actuator_y_size/2)+wheel_length/2} 0.0" rpy="0 0 0" />
 	</xacro:igor_wheel>
@@ -124,5 +124,5 @@
 		<origin xyz="${0} ${actuator_y_size-0.0038} -${lower_leg_length+actuator_z_size/2.5}" rpy="0 0 0" />
 	</xacro:igor_actuator>
-	<xacro:igor_wheel prefix="L" flip="1" reflect="1" damping="${0.25}">
+	<xacro:igor_wheel prefix="L" flip="1" reflect="1" damping="${0.17}" static_friction="0.0011">
 		<origin xyz="${0} ${(actuator_y_size/2)+wheel_length/2} 0.0" rpy="0 0 0" />
 	</xacro:igor_wheel>

File: urdf/lowerleg.urdf.xacro (robot description, xacro)
@@ -27,5 +27,5 @@
 			<parent link="${prefix}_kneeActuator"/>
 			<child  link="${prefix}_lowerleg"/>
-			<limit effort="15" lower="0" upper="0" velocity="10"/>
+			<limit effort="15" lower="${-0.65}" upper="${-0.65}" velocity="10"/>
 			<axis xyz="0 1 0"/>
 			<dynamics damping="0.1"/>

File: urdf/upperleg.urdf.xacro (robot description, xacro)
@@ -29,5 +29,5 @@
 			<parent link="${prefix}_baseActuator"/>
 			<child  link="${prefix}_upperleg"/>
-			<limit effort="${15}" lower="-0" upper="0" velocity="10"/>
+			<limit effort="${15}" lower="${1.9-M_PI/2}" upper="${1.9-M_PI/2}" velocity="10"/>
 			<axis xyz="0 1 0"/>
 			<dynamics damping="0.1"/>

File: urdf/wheel.urdf.xacro (robot description, xacro)
@@ -1,5 +1,5 @@
 <?xml version="1.0"?>
 <robot xmlns:xacro="http://ros.org/wiki/xacro" name="igor_wheel">
-	<xacro:macro name="igor_wheel" params="prefix flip reflect damping *joint_pose">
+	<xacro:macro name="igor_wheel" params="prefix flip reflect damping static_friction *joint_pose">
 		<link name="${prefix}_wheel">
 			<visual>
@@ -39,7 +39,7 @@
 			<parent link="${prefix}_wheelActuator"/>
 			<child  link="${prefix}_wheel"/>
-			<limit effort="3" velocity="20"/>  <!-- effort limit in N (prismatic) or N.m (revolute), Velocity limit in m/s or rad/s -->
+			<limit effort="3" velocity="12"/>  <!-- effort limit in N (prismatic) or N.m (revolute), Velocity limit in m/s or rad/s -->
 			<axis xyz="0 1 0"/>
-			<dynamics damping="${damping}" friction="0.0011"/>
+			<dynamics damping="${damping}" friction="${static_friction}"/>
 		</joint>
     		<!--transmission name="Diff_${prefix}_wheel_trans">
