Commit message: Manipulator control added

File: urdf/Igor_armed.urdf.xacro (robot description, xacro)
@@ -125,14 +125,18 @@
 		<origin xyz="${0} ${0} ${base_z_size/2 + 0.015}" rpy="${M_PI/2} 0 0" />
 	</xacro:igor_actuator>
-	<xacro:arm prefix="Upper" reflect="1" flip="0">
-		<origin xyz="${0} ${actuator_y_size/2+lower_leg_radius} 0.0" rpy="0 ${M_PI/2} ${M_PI}" />
+	<xacro:arm prefix="Upper" reflect="-1" flip="0">
+		<origin xyz="${0} ${actuator_y_size/2+lower_leg_radius} ${0.0}" rpy="${-M_PI/2} ${0} ${0}" />
 	</xacro:arm>
 	<!--Forearm-->
 	<xacro:igor_actuator prefix="Fore_arm" reflect="1" parent_link="Upper_arm" flip="1">
-		<origin xyz="${0} ${actuator_y_size/1.2} -${lower_leg_length + actuator_z_size/2.3}" rpy="${0} ${M_PI/2} 0" />
-	</xacro:igor_actuator>
-	<xacro:arm prefix="Fore" reflect="1" flip="0">
-		<origin xyz="${0} ${actuator_y_size/2+lower_leg_radius} 0.0" rpy="0 ${M_PI/2} ${M_PI}" />
+		<origin xyz="${lower_leg_length + actuator_z_size/2.3} ${0} -${actuator_y_size/1.2}" rpy="${M_PI/2} ${0} 0" />
+	</xacro:igor_actuator>
+	<xacro:arm prefix="Fore" reflect="1" flip="1">
+		<origin xyz="${0} -${actuator_y_size/2+lower_leg_radius} 0.0" rpy="${-M_PI/2} ${0} ${0}" />
 	</xacro:arm>
+	<!--Endeffector-->
+	<xacro:igor_actuator prefix="Endeffector" reflect="1" parent_link="Fore_arm" flip="1">
+		<origin xyz="${lower_leg_length + actuator_z_size/2.3} ${0} ${actuator_y_size/1.2}" rpy="${M_PI/2} ${0} 0" />
+	</xacro:igor_actuator>
 	<!--Robot Center Dummy-->
 	<link name="robot_center_link">

File: urdf/arm.urdf.xacro (robot description, xacro)
@@ -4,5 +4,5 @@
 		<link name="${prefix}_arm">
 			<visual>
-				<origin rpy="${M_PI/2} ${M_PI/2} ${flip*M_PI}" xyz="${reflect*-2.5*lower_leg_radius} ${reflect*2*lower_leg_radius} ${actuator_z_size/1.5}"/>
+				<origin rpy="${flip*M_PI} ${0} ${0}" xyz="-${actuator_z_size/1.5} ${reflect*2.5*lower_leg_radius}  ${reflect*2*lower_leg_radius}"/>
 				<geometry>
 					<mesh filename="package://igor/meshes/lowerLeg.STL" scale="0.001 0.001 0.001"/>
@@ -11,5 +11,5 @@
 		    	</visual>
 			<collision>
-				<origin rpy="0.0 0.0 0.0" xyz="0.0 0.0 -${lower_leg_length/2}"/>
+				<origin rpy="0.0 ${M_PI/2} 0.0" xyz="${lower_leg_length/2} 0.0 ${0}"/>
 				<geometry>
 					<cylinder radius="${lower_leg_radius}" length="${lower_leg_length}" /> <!-- Actual dimensions -->
@@ -17,5 +17,5 @@
 		    	</collision>
 	    		<inertial>
-				<origin rpy="0.0 0.0 0.0" xyz="0.0 0.0 -${lower_leg_length/2}"/>
+				<origin rpy="0.0 ${M_PI/2} 0.0" xyz="${lower_leg_length/2} 0.0 ${0}"/>
 	      			<mass value="0.2"/>
 	      			<inertia ixx="0.001521" ixy="0.00" ixz="0.00" iyy="0.001521" iyz="0.000" izz="4.2E-05"/>
@@ -26,6 +26,6 @@
 			<parent link="${prefix}_armActuator"/>
 			<child  link="${prefix}_arm"/>
-			<limit effort="5" lower="${0}" upper="${0}" velocity="10"/>
-			<axis xyz="0 1 0"/>
+			<limit effort="5" lower="${-2}" upper="${2}" velocity="10"/>
+			<axis xyz="0 0 1"/>
 			<dynamics damping="0.1"/>
 		</joint>
